File: Eagle-Conversion/Example_Board_To_Convert.brd (EAGLE design)
At the start: 30.5 x 25.4 mm, 33 parts, among them J2 SMD, J3 PTH, J4 SMD, J6 SPI, U2 BNO080

Commit message: Fixed some bugs and added possibility to turn of fiducial referencing and added a third mark to Nathans PCB example
Parts:
- added JP1: FIDUCIALUFIDUCIAL, SparkFun:MICRO-FIDUCIAL
Changed lines of the file:
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@@
 <element name="J5" library="SparkFun-Connectors" package="1X01_NO_SILK" value="" x="1.27" y="7.62"/>
 <element name="J8" library="SparkFun-Connectors" package="1X02_NO_SILK" value="" x="8.89" y="1.27" rot="R180"/>
+<element name="JP1" library="SparkFun" package="MICRO-FIDUCIAL" value="FIDUCIALUFIDUCIAL" x="29.718" y="24.638"/>
 </elements>
 <signals>
